Commit message: 수업내용

File: mastering_ros_robot_description_pkg/urdf/seven_dof_arm.xacro (robot description, xacro)
@@ -144,5 +144,5 @@
   </link>
   <gazebo reference="shoulder_pan_link">
-    <material>Gazebo/Red</material>
+    <material>Gazebo/Blue</material>
   </gazebo>
   <joint name="shoulder_pitch_joint" type="revolute">
@@ -231,5 +231,5 @@
   </link>
   <gazebo reference="elbow_pitch_link">
-    <material>Gazebo/Red</material>
+    <material>Gazebo/Blue</material>
   </gazebo>
   <joint name="wrist_roll_joint" type="revolute">
@@ -320,5 +320,5 @@
   </link>
   <gazebo reference="gripper_roll_link">
-    <material>Gazebo/Red</material>
+    <material>Gazebo/Blue</material>
   </gazebo>
   <joint name="finger_joint1" type="prismatic">
