Commit message: day7초기 코드

File: mastering_ros_robot_description_pkg/urdf/diff_wheeled_robot_with_laser.xacro (robot description, xacro)
@@ -2,5 +2,5 @@
 <robot name="differential_wheeled_robot" xmlns:xacro="http://ros.org/wiki/xacro">
   <xacro:include filename="$(find mastering_ros_robot_description_pkg)/urdf/wheel.urdf.xacro" />
-    <!-- Defining the colors used in this robot -->
+	<!-- Defining the colors used in this robot -->
   <material name="Black">
     <color rgba="0.0 0.0 0.0 1.0"/>
@@ -104,5 +104,5 @@
       <origin xyz="0 0.02 0" rpy="${M_PI/2} 0 0" />
       <geometry>
-                <sphere radius="${caster_f_radius}" />
+				<sphere radius="${caster_f_radius}" />
       </geometry>
       <material name="Black" />
@@ -110,5 +110,5 @@
     <collision>
       <geometry>
-                <sphere radius="${caster_f_radius}" />
+				<sphere radius="${caster_f_radius}" />
       </geometry>
     <origin xyz="0 0.02 0" rpy="${M_PI/2} 0 0" />
@@ -122,5 +122,5 @@
     </inertial>
   </link>
-    <joint name="caster_front_joint" type="fixed">
+	<joint name="caster_front_joint" type="fixed">
     <parent link="base_link"/>
     <child link="caster_front_link"/>
@@ -134,5 +134,5 @@
     <origin xyz="0.02 0.02 0 " rpy="${M_PI/2} 0 0" />
     <geometry>
-            <sphere radius="${caster_b_radius}" />
+			<sphere radius="${caster_b_radius}" />
     </geometry>
     <material name="Black" />
@@ -140,5 +140,5 @@
   <collision>
     <geometry>
-            <sphere radius="${caster_b_radius}" />
+			<sphere radius="${caster_b_radius}" />
      </geometry>
      <origin xyz="0 0.02 0 " rpy="${M_PI/2} 0 0" />
@@ -161,29 +161,29 @@
   </gazebo>
   <xacro:wheel fb="front" lr="right" parent="base_link" translateX="0" translateY="-0.5" flipY="1"/>
-    <xacro:wheel fb="front" lr="left" parent="base_link" translateX="0" translateY="0.5" flipY="1"/>
-    <gazebo>
-      <plugin name="differential_drive_controller" filename="libgazebo_ros_diff_drive.so">
-        <legacyMode>true</legacyMode>
-        <rosDebugLevel>Debug</rosDebugLevel>
-        <publishWheelTF>false</publishWheelTF>
-        <robotNamespace>/</robotNamespace>
-        <publishTf>1</publishTf>
-        <publishWheelJointState>false</publishWheelJointState>
-        <alwaysOn>true</alwaysOn>
-        <updateRate>100.0</updateRate>
-        <leftJoint>front_left_wheel_joint</leftJoint>
-        <rightJoint>front_right_wheel_joint</rightJoint>
-        <wheelSeparation>${2*base_radius}</wheelSeparation>
-        <wheelDiameter>${2*wheel_radius}</wheelDiameter>
-        <broadcastTF>1</broadcastTF>
-        <wheelTorque>30</wheelTorque>
-        <wheelAcceleration>1.8</wheelAcceleration>
-        <commandTopic>cmd_vel</commandTopic>
-        <odometryFrame>odom</odometryFrame>
-        <odometryTopic>odom</odometryTopic>
-        <robotBaseFrame>base_footprint</robotBaseFrame>
+	<xacro:wheel fb="front" lr="left" parent="base_link" translateX="0" translateY="0.5" flipY="1"/>
+	<gazebo>
+  	<plugin name="differential_drive_controller" filename="libgazebo_ros_diff_drive.so">
+	    <legacyMode>true</legacyMode>
+	    <rosDebugLevel>Debug</rosDebugLevel>
+	    <publishWheelTF>false</publishWheelTF>
+	    <robotNamespace>/</robotNamespace>
+	    <publishTf>1</publishTf>
+	    <publishWheelJointState>false</publishWheelJointState>
+	    <alwaysOn>true</alwaysOn>
+	    <updateRate>100.0</updateRate>
+	    <leftJoint>front_left_wheel_joint</leftJoint>
+	    <rightJoint>front_right_wheel_joint</rightJoint>
+	    <wheelSeparation>${2*base_radius}</wheelSeparation>
+	    <wheelDiameter>${2*wheel_radius}</wheelDiameter>
+	    <broadcastTF>1</broadcastTF>
+	    <wheelTorque>30</wheelTorque>
+	    <wheelAcceleration>1.8</wheelAcceleration>
+	    <commandTopic>cmd_vel</commandTopic>
+	    <odometryFrame>odom</odometryFrame>
+	    <odometryTopic>odom</odometryTopic>
+	    <robotBaseFrame>base_footprint</robotBaseFrame>
    </plugin>
   </gazebo>
-  <link name="laser_link">
+	<link name="laser_link">
     <visual>
       <origin xyz="0 0 0" rpy="0 0 0" />
@@ -194,7 +194,6 @@
     </visual>
   </link>
-  <!-- Step 3: 센서를 중앙(x=0), 낮은 높이로 배치 + 360° 스캔 -->
   <joint name="hokuyo_joint" type="fixed">
-    <origin xyz="0 0 ${base_height+hokuyo_size/4}" rpy="0 0 0" />
+    <origin xyz="${base_radius - hokuyo_size/2} 0 ${base_height+hokuyo_size/4}" rpy="0 0 0" />
     <parent link="base_link"/>
     <child link="laser_link" />
@@ -204,5 +203,5 @@
     <turnGravityOff>false</turnGravityOff>
     <sensor type="ray" name="head_hokuyo_sensor">
-      <pose>0 0 0 0 0 0</pose>
+      <pose>${hokuyo_size/2} 0 0 0 0 0</pose>
       <visualize>true</visualize>
       <update_rate>40</update_rate>
@@ -212,6 +211,6 @@
             <samples>720</samples>
             <resolution>1</resolution>
-            <min_angle>-3.14159</min_angle>
-            <max_angle>3.14159</max_angle>
+            <min_angle>-1.570796</min_angle>
+            <max_angle>1.570796</max_angle>
           </horizontal>
         </scan>
